File: hardware/numpad/goboard-numpad.kicad_sch (KiCad schematic)
At the start: 0 parts

Commit message: Add first schematic for the numpad
Parts:
- added J?: Conn_01x07_Male, symbol Connector:Conn_01x07_Male
- added R?: R, symbol Device:R
Connections:
- new net: J?.5 (Pin_5), R?.2
- new net GND: J?.7 (Pin_7)
- new net Keys/165_~CE: J?.3 (Pin_3)
- new net Keys/165_~PL: J?.4 (Pin_4)
- new net Keys/SPI_MOSI: J?.1 (Pin_1)
- new net Keys/SPI_SCK: J?.2 (Pin_2)
- new net VCC: J?.6 (Pin_6), R?.1
Other:
- added sheet Keys (keys.kicad_sch)
- note added: "TODO: Better way to detect if the numpad is attached?"
