File: hardware/main/mcu.kicad_sch (KiCad schematic)
At the start: 0 parts

Commit message: Add connector to the numpad to the schematic
Parts:
- added C3: 100nF, symbol Device:C
- added D45: Power, symbol Device:LED
- added D46: Caps Lock, symbol Device:LED
- added D47: Scroll Lock, symbol Device:LED
- added R4, R5, R6: 47, symbol Device:R
- added U1: Holyiot-18010-NRF52840, footprints:Holyiot-18010-NRF52840, symbol symbols:Holyiot-18010-NRF52840
Connections:
- new net: D47.2 (A), R6.1
- new net: D45.2 (A), R4.1
- new net: D46.2 (A), R5.1
- new net D+: U1.24 (D+)
- new net D-: U1.23 (D-)
- new net GND: C3.2
- new net VCC_SW: C3.1, U1.14 (VDD_nRF)
- no-connect marks 0 -> 18
Changed lines of the file:
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@@
 (kicad_sch (version 20201015) (generator eeschema)
   (paper "A4")
+  (junction (at 139.7 29.21) (diameter 1.016) (color 0 0 0 0))
+  (no_connect (at 152.4 110.49))
+  (no_connect (at 152.4 85.09))
+  (no_connect (at 152.4 87.63))
+  (no_connect (at 152.4 72.39))
+  (no_connect (at 152.4 77.47))
+  (no_connect (at 127 69.85))
+  (no_connect (at 152.4 107.95))
+  (no_connect (at 152.4 105.41))
+  (no_connect (at 152.4 64.77))
+  (no_connect (at 152.4 59.69))
+  (no_connect (at 152.4 82.55))
+  (no_connect (at 127 62.23))
+  (no_connect (at 127 67.31))
+  (no_connect (at 127 80.01))
+  (no_connect (at 152.4 113.03))
+  (no_connect (at 152.4 95.25))
+  (no_connect (at 152.4 80.01))
+  (no_connect (at 127 85.09))
+  (wire (pts (xy 116.84 29.21) (xy 139.7 29.21))
+    (stroke (width 0) (type solid) (color 0 0 0 0))
+  )
+  (wire (pts (xy 116.84 36.83) (xy 116.84 39.37))
+    (stroke (width 0) (type solid) (color 0 0 0 0))
+  )
+  (wire (pts (xy 124.46 100.33) (xy 127 100.33))
+    (stroke (width 0) (type solid) (color 0 0 0 0))
+  )
+  (wire (pts (xy 124.46 102.87) (xy 127 102.87))
+    (stroke (width 0) (type solid) (color 0 0 0 0))
+  )
+  (wire (pts (xy 139.7 29.21) (xy 139.7 25.4))
+    (stroke (width 0) (type solid) (color 0 0 0 0))
+  )
+  (wire (pts (xy 139.7 44.45) (xy 139.7 29.21))
+    (stroke (width 0) (type solid) (color 0 0 0 0))
+  )
+  (wire (pts (xy 229.87 68.58) (xy 232.41 68.58))
+    (stroke (width 0) (type solid) (color 0 0 0 0))
+  )
+  (wire (pts (xy 229.87 78.74) (xy 232.41 78.74))
+    (stroke (width 0) (type solid) (color 0 0 0 0))
+  )
+  (wire (pts (xy 229.87 88.9) (xy 232.41 88.9))
+    (stroke (width 0) (type solid) (color 0 0 0 0))
+  )
+  (hierarchical_label "D-" (shape input) (at 124.46 100.33 180)
+    (effects (font (size 1.27 1.27)) (justify right))
+  )
+  (hierarchical_label "D+" (shape input) (at 124.46 102.87 180)
+    (effects (font (size 1.27 1.27)) (justify right))
+  )
+  (hierarchical_label "VCC_SW" (shape input) (at 139.7 25.4 90)
+    (effects (font (size 1.27 1.27)) (justify left))
+  )
+  (symbol (lib_id "power:GND") (at 116.84 39.37 0) (unit 1)
+    (in_bom yes) (on_board yes)
+    (property "Reference" "#PWR0109" (id 0) (at 116.84 45.72 0)
+      (effects (font (size 1.27 1.27)) hide)
+    )
+    (property "Value" "GND" (id 1) (at 118.11 44.45 0))
+    (property "Footprint" "" (id 2) (at 116.84 39.37 0)
+      (effects (font (size 1.27 1.27)) hide)
+    )
+    (property "Datasheet" "" (id 3) (at 116.84 39.37 0)
+      (effects (font (size 1.27 1.27)) hide)
+    )
+  )
+  (symbol (lib_id "Device:R") (at 236.22 68.58 90) (unit 1)
+    (in_bom yes) (on_board yes)
+    (property "Reference" "R4" (id 0) (at 236.22 62.23 90))
+    (property "Value" "47" (id 1) (at 236.22 64.77 90))
+    (property "Footprint" "" (id 2) (at 236.22 70.358 90)
+      (effects (font (size 1.27 1.27)) hide)
+    )
+    (property "Datasheet" "~" (id 3) (at 236.22 68.58 0)
+      (effects (font (size 1.27 1.27)) hide)
+    )
+  )
+  (symbol (lib_id "Device:R") (at 236.22 78.74 90) (unit 1)
+    (in_bom yes) (on_board yes)
+    (property "Reference" "R5" (id 0) (at 236.22 72.39 90))
+    (property "Value" "47" (id 1) (at 236.22 74.93 90))
+    (property "Footprint" "" (id 2) (at 236.22 80.518 90)
+      (effects (font (size 1.27 1.27)) hide)
+    )
+    (property "Datasheet" "~" (id 3) (at 236.22 78.74 0)
+      (effects (font (size 1.27 1.27)) hide)
+    )
+  )
+  (symbol (lib_id "Device:R") (at 236.22 88.9 90) (unit 1)
+    (in_bom yes) (on_board yes)
+    (property "Reference" "R6" (id 0) (at 236.22 82.55 90))
+    (property "Value" "47" (id 1) (at 236.22 85.09 90))
+    (property "Footprint" "" (id 2) (at 236.22 90.678 90)
+      (effects (font (size 1.27 1.27)) hide)
+    )
+    (property "Datasheet" "~" (id 3) (at 236.22 88.9 0)
+      (effects (font (size 1.27 1.27)) hide)
+    )
+  )
+  (symbol (lib_id "Device:LED") (at 226.06 68.58 0) (unit 1)
+    (in_bom yes) (on_board yes)
+    (property "Reference" "D45" (id 0) (at 226.06 62.23 0))
+    (property "Value" "Power" (id 1) (at 226.06 64.77 0))
+    (property "Footprint" "" (id 2) (at 226.06 68.58 0)
+      (effects (font (size 1.27 1.27)) hide)
+    )
+    (property "Datasheet" "~" (id 3) (at 226.06 68.58 0)
+      (effects (font (size 1.27 1.27)) hide)
+    )
+  )
+  (symbol (lib_id "Device:LED") (at 226.06 78.74 0) (unit 1)
+    (in_bom yes) (on_board yes)
+    (property "Reference" "D46" (id 0) (at 226.06 72.39 0))
+    (property "Value" "Caps Lock" (id 1) (at 226.06 74.93 0))
+    (property "Footprint" "" (id 2) (at 226.06 78.74 0)
+      (effects (font (size 1.27 1.27)) hide)
+    )
+    (property "Datasheet" "~" (id 3) (at 226.06 78.74 0)
+      (effects (font (size 1.27 1.27)) hide)
+    )
+  )
+  (symbol (lib_id "Device:LED") (at 226.06 88.9 0) (unit 1)
+    (in_bom yes) (on_board yes)
+    (property "Reference" "D47" (id 0) (at 226.06 82.55 0))
+    (property "Value" "Scroll Lock" (id 1) (at 226.06 85.09 0))
+    (property "Footprint" "" (id 2) (at 226.06 88.9 0)
+      (effects (font (size 1.27 1.27)) hide)
+    )
+    (property "Datasheet" "~" (id 3) (at 226.06 88.9 0)
+      (effects (font (size 1.27 1.27)) hide)
+    )
+  )
+  (symbol (lib_id "Device:C") (at 116.84 33.02 0) (unit 1)
+    (in_bom yes) (on_board yes)
+    (property "Reference" "C3" (id 0) (at 120.65 31.75 0)
+      (effects (font (size 1.27 1.27)) (justify left))
+    )
+    (property "Value" "100nF" (id 1) (at 120.65 34.29 0)
+      (effects (font (size 1.27 1.27)) (justify left))
+    )
+    (property "Footprint" "" (id 2) (at 117.8052 36.83 0)
+      (effects (font (size 1.27 1.27)) hide)
+    )
+    (property "Datasheet" "~" (id 3) (at 116.84 33.02 0)
+      (effects (font (size 1.27 1.27)) hide)
+    )
+  )
+  (symbol (lib_id "symbols:Holyiot-18010-NRF52840") (at 139.7 86.36 0) (unit 1)
+    (in_bom yes) (on_board yes)
+    (property "Reference" "U1" (id 0) (at 139.7 39.37 0))
+    (property "Value" "Holyiot-18010-NRF52840" (id 1) (at 139.7 41.91 0))
+    (property "Footprint" "footprints:Holyiot-18010-NRF52840" (id 2) (at 130.81 45.72 0)
+      (effects (font (size 1.27 1.27)) hide)
+    )
+    (property "Datasheet" "http://www.holyiot.com/tp/2019042516322180424.pdf" (id 3) (at 130.81 45.72 0)
+      (effects (font (size 1.27 1.27)) hide)
+    )
+  )
 )
