File: hardware/main/goboard-main.kicad_pcb (KiCad board)
At the start: 2 copper layers, 309.6 x 123.8 mm, 86 parts, among them SW1 Esc, SW10 a, SW11 \, SW12 Fn, SW13 F2, SW14 2, SW15 w, SW16 s, SW17 z, SW18 Tux, SW19 F3, SW2 F1, SW20 3, SW21 e, SW22 d, SW23 c, SW24 Alt, SW25 F4, SW26 4, SW27 r, SW28 f, SW29 v, SW3 tilde, SW31 F5, SW32 5, SW33 t, SW34 g, SW35 b, SW36 F6, SW37 6, SW38 y, SW39 h, SW4 Tab, SW40 n, SW41 F7, SW42 7, SW43 u, SW44 j, SW45 m, SW46 Space, SW47 F8, SW48 8, SW49 i, SW5 Caps Lock, SW50 k, SW51 ,, SW52 F9, SW53 9, SW54 o, SW55 l, SW56 ., SW57 F10, SW58 0, SW59 p, SW6 Shift, SW60 ;, SW61 /, SW62 Alt Gr, SW63 F11, SW64 -, SW65 [, SW66 ', SW67 Menu, SW68 F12, SW69 =, SW7 Ctrl, SW70 ], SW71 \, SW72 Shift, SW73 Ctrl, SW74 Print, SW75 Backspace, SW76 Enter, SW77 Left, SW78 Scroll Lock, SW79 Up, SW8 1, SW80 Down, SW81 Pause, SW82 INS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

Commit message: Implement the key matrix on the PCB
Parts:
- removed SW11: \, footprints:SW_Cherry_MX_1.00u_PCB
- added D1: BAT54C, Package_TO_SOT_SMD:SOT-23, B.Cu at (46.2, 37.0)
- added D10: BAT54C, Package_TO_SOT_SMD:SOT-23, B.Cu at (94.8, 94.3)
- added D11: BAT54C, Package_TO_SOT_SMD:SOT-23, B.Cu at (88.0, 113.3)
- added D12: BAT54C, Package_TO_SOT_SMD:SOT-23, B.Cu at (88.0, 129.6)
- added D13: BAT54C, Package_TO_SOT_SMD:SOT-23, B.Cu at (121.3, 37.1)
- added D14: BAT54C, Package_TO_SOT_SMD:SOT-23, B.Cu at (121.3, 56.0)
- added D15: BAT54C, Package_TO_SOT_SMD:SOT-23, B.Cu at (130.8, 75.2)
- added D16: BAT54C, Package_TO_SOT_SMD:SOT-23, B.Cu at (135.6, 94.2)
- added D17: BAT54C, Package_TO_SOT_SMD:SOT-23, B.Cu at (126.0, 113.3)
- added D18: BAT54C, Package_TO_SOT_SMD:SOT-23, B.Cu at (159.4, 37.1)
- added D19: BAT54C, Package_TO_SOT_SMD:SOT-23, B.Cu at (159.4, 56.1)
- added D2: BAT54C, Package_TO_SOT_SMD:SOT-23, B.Cu at (46.3, 56.2)
- added D20: BAT54C, Package_TO_SOT_SMD:SOT-23, B.Cu at (168.9, 75.2)
- added D21: BAT54C, Package_TO_SOT_SMD:SOT-23, B.Cu at (173.7, 94.2)
- added D22: BAT54C, Package_TO_SOT_SMD:SOT-23, B.Cu at (164.1, 113.3)
- added D24: BAT54C, Package_TO_SOT_SMD:SOT-23, B.Cu at (197.4, 37.1)
- added D25: BAT54C, Package_TO_SOT_SMD:SOT-23, B.Cu at (197.5, 56.1)
- added D26: BAT54C, Package_TO_SOT_SMD:SOT-23, B.Cu at (207.0, 75.2)
- added D27: BAT54C, Package_TO_SOT_SMD:SOT-23, B.Cu at (211.8, 94.2)
- added D28: BAT54C, Package_TO_SOT_SMD:SOT-23, B.Cu at (202.2, 113.3)
- added D29: BAT54C, Package_TO_SOT_SMD:SOT-23, B.Cu at (235.6, 37.1)
- added D3: BAT54C, Package_TO_SOT_SMD:SOT-23, B.Cu at (46.1, 75.2)
- added D30: BAT54C, Package_TO_SOT_SMD:SOT-23, B.Cu at (235.6, 56.1)
- added D31: BAT54C, Package_TO_SOT_SMD:SOT-23, B.Cu at (245.1, 75.2)
- added D32: BAT54C, Package_TO_SOT_SMD:SOT-23, B.Cu at (249.9, 94.2)
- added D33: BAT54C, Package_TO_SOT_SMD:SOT-23, B.Cu at (240.4, 113.2)
- added D34: BAT54C, Package_TO_SOT_SMD:SOT-23, B.Cu at (237.4, 132.5)
- added D35: BAT54C, Package_TO_SOT_SMD:SOT-23, B.Cu at (273.7, 37.1)
- added D36: BAT54C, Package_TO_SOT_SMD:SOT-23, B.Cu at (271.3, 56.1)
- added D37: BAT54C, Package_TO_SOT_SMD:SOT-23, B.Cu at (280.9, 77.8)
- added D38: BAT54C, Package_TO_SOT_SMD:SOT-23, B.Cu at (285.6, 94.2)
- added D39: BAT54C, Package_TO_SOT_SMD:SOT-23, B.Cu at (289.8, 113.3)
- added D4: BAT54C, Package_TO_SOT_SMD:SOT-23, B.Cu at (46.1, 91.9)
- added D40: BAT54C, Package_TO_SOT_SMD:SOT-23, B.Cu at (273.7, 132.3)
- added D41: BAT54C, Package_TO_SOT_SMD:SOT-23, B.Cu at (311.8, 37.1)
- added D42: BAT54C, Package_TO_SOT_SMD:SOT-23, B.Cu at (318.6, 56.1)
- added D43: BAT54C, Package_TO_SOT_SMD:SOT-23, B.Cu at (311.8, 113.3)
- added D44: BAT54C, Package_TO_SOT_SMD:SOT-23, B.Cu at (311.8, 132.3)
- added D5: BAT54C, Package_TO_SOT_SMD:SOT-23, B.Cu at (47.0, 113.3)
- added D6: BAT54C, Package_TO_SOT_SMD:SOT-23, B.Cu at (47.0, 132.3)
- added D7: BAT54C, Package_TO_SOT_SMD:SOT-23, B.Cu at (83.2, 37.1)
- added D8: BAT54C, Package_TO_SOT_SMD:SOT-23, B.Cu at (83.2, 56.1)
- added D9: BAT54C, Package_TO_SOT_SMD:SOT-23, B.Cu at (92.8, 75.2)
- added U1: 74LV595, Package_SO:TSSOP-16_4.4x5mm_P0.65mm, B.Cu at (289.7, 68.0)
- added U2: 74LV165, Package_SO:TSSOP-16_4.4x5mm_P0.65mm, F.Cu at (289.8, 61.2)
- added U3: 74LV165, Package_SO:TSSOP-16_4.4x5mm_P0.65mm, B.Cu at (260.3, 48.4)
Connections:
- SW10 pad 2: Net-(SW10-Pad2) -> Net-(SW2-Pad2)
- SW12 pad 2: Net-(SW12-Pad2) -> Net-(SW2-Pad2)
- SW14 pad 2: Net-(SW14-Pad2) -> Net-(SW13-Pad2)
- SW15 pad 2: Net-(SW15-Pad2) -> Net-(SW13-Pad2)
- SW16 pad 2: Net-(SW16-Pad2) -> Net-(SW13-Pad2)
- SW17 pad 2: Net-(SW17-Pad2) -> Net-(SW13-Pad2)
- SW18 pad 2: Net-(SW18-Pad2) -> Net-(SW2-Pad2)
- SW20 pad 2: Net-(SW20-Pad2) -> Net-(SW19-Pad2)
- SW21 pad 2: Net-(SW21-Pad2) -> Net-(SW19-Pad2)
- SW22 pad 2: Net-(SW22-Pad2) -> Net-(SW19-Pad2)
- SW23 pad 2: Net-(SW23-Pad2) -> Net-(SW27-Pad2)
- SW24 pad 2: Net-(SW24-Pad2) -> Net-(SW13-Pad2)
- SW25 pad 2: Net-(SW25-Pad2) -> Net-(SW27-Pad2)
- SW26 pad 2: Net-(SW26-Pad2) -> Net-(SW27-Pad2)
- SW28 pad 2: Net-(SW28-Pad2) -> Net-(SW27-Pad2)
- SW29 pad 2: Net-(SW29-Pad2) -> Net-(SW32-Pad2)
- SW3 pad 2: Net-(SW3-Pad2) -> Net-(SW1-Pad2)
- SW31 pad 2: Net-(SW31-Pad2) -> Net-(SW32-Pad2)
- SW33 pad 2: Net-(SW33-Pad2) -> Net-(SW32-Pad2)
- SW34 pad 2: Net-(SW34-Pad2) -> Net-(SW32-Pad2)
- SW35 pad 2: Net-(SW35-Pad2) -> Net-(SW38-Pad2)
- SW36 pad 2: Net-(SW36-Pad2) -> Net-(SW38-Pad2)
- SW37 pad 2: Net-(SW37-Pad2) -> Net-(SW38-Pad2)
- SW39 pad 2: Net-(SW39-Pad2) -> Net-(SW38-Pad2)
- SW4 pad 2: Net-(SW4-Pad2) -> Net-(SW1-Pad2)
- SW40 pad 2: Net-(SW40-Pad2) -> Net-(SW43-Pad2)
- SW41 pad 2: Net-(SW41-Pad2) -> Net-(SW43-Pad2)
- SW42 pad 2: Net-(SW42-Pad2) -> Net-(SW43-Pad2)
- SW44 pad 2: Net-(SW44-Pad2) -> Net-(SW43-Pad2)
- SW45 pad 2: Net-(SW45-Pad2) -> Net-(SW49-Pad2)
- SW46 pad 2: Net-(SW46-Pad2) -> Net-(SW38-Pad2)
- SW47 pad 2: Net-(SW47-Pad2) -> Net-(SW49-Pad2)
- SW48 pad 2: Net-(SW48-Pad2) -> Net-(SW49-Pad2)
- SW5 pad 2: Net-(SW5-Pad2) -> Net-(SW1-Pad2)
- SW50 pad 2: Net-(SW50-Pad2) -> Net-(SW49-Pad2)
- SW51 pad 2: Net-(SW51-Pad2) -> Net-(SW54-Pad2)
- SW52 pad 2: Net-(SW52-Pad2) -> Net-(SW54-Pad2)
- SW53 pad 2: Net-(SW53-Pad2) -> Net-(SW54-Pad2)
- SW55 pad 2: Net-(SW55-Pad2) -> Net-(SW54-Pad2)
- SW56 pad 2: Net-(SW56-Pad2) -> Net-(SW62-Pad2)
- SW57 pad 2: Net-(SW57-Pad2) -> Net-(SW62-Pad2)
- SW58 pad 2: Net-(SW58-Pad2) -> Net-(SW62-Pad2)
- SW59 pad 2: Net-(SW59-Pad2) -> Net-(SW62-Pad2)
- SW6 pad 2: Net-(SW6-Pad2) -> Net-(SW1-Pad2)
- SW60 pad 2: Net-(SW60-Pad2) -> Net-(SW62-Pad2)
- SW61 pad 2: Net-(SW61-Pad2) -> Net-(SW67-Pad2)
- SW63 pad 2: Net-(SW63-Pad2) -> Net-(SW67-Pad2)
- SW64 pad 2: Net-(SW64-Pad2) -> Net-(SW67-Pad2)
- SW65 pad 2: Net-(SW65-Pad2) -> Net-(SW67-Pad2)
- SW66 pad 2: Net-(SW66-Pad2) -> Net-(SW67-Pad2)
- SW68 pad 2: Net-(SW68-Pad2) -> Net-(SW70-Pad2)
- SW69 pad 2: Net-(SW69-Pad2) -> Net-(SW70-Pad2)
- SW7 pad 2: Net-(SW7-Pad2) -> Net-(SW1-Pad2)
- SW71 pad 2: Net-(SW71-Pad2) -> Net-(SW70-Pad2)
- SW72 pad 2: Net-(SW72-Pad2) -> Net-(SW70-Pad2)
- SW73 pad 2: Net-(SW73-Pad2) -> Net-(SW70-Pad2)
- SW74 pad 2: Net-(SW74-Pad2) -> Net-(SW75-Pad2)
- SW76 pad 2: Net-(SW76-Pad2) -> Net-(SW75-Pad2)
- SW77 pad 2: Net-(SW77-Pad2) -> Net-(SW75-Pad2)
- SW79 pad 2: Net-(SW79-Pad2) -> Net-(SW78-Pad2)
- SW8 pad 2: Net-(SW8-Pad2) -> Net-(SW2-Pad2)
- SW80 pad 2: Net-(SW80-Pad2) -> Net-(SW78-Pad2)
- SW82 pad 2: Net-(SW82-Pad2) -> Net-(SW81-Pad2)
- SW83 pad 2: Net-(SW83-Pad2) -> Net-(SW78-Pad2)
- SW84 pad 2: Net-(SW84-Pad2) -> Net-(SW81-Pad2)
- SW85 pad 2: Net-(SW85-Pad2) -> Net-(SW81-Pad2)
- SW86 pad 2: Net-(SW86-Pad2) -> Net-(SW81-Pad2)
- SW87 pad 2: Net-(SW87-Pad2) -> Net-(SW19-Pad2)
- SW9 pad 2: Net-(SW9-Pad2) -> Net-(SW2-Pad2)
Routing:
- net Net-(U1-Pad2): track 0.00 -> 339.6 mm, vias 0 -> 4
- net Net-(U1-Pad15): track 0.00 -> 312.6 mm, vias 0 -> 2
- net Net-(U1-Pad1): track 0.00 -> 308.2 mm, vias 0 -> 4
- net Net-(D14-Pad3): track 0.00 -> 296.3 mm
- net Net-(U1-Pad3): track 0.00 -> 277.1 mm, vias 0 -> 2
- net Net-(D15-Pad3): track 0.00 -> 253.7 mm
- net Net-(SW78-Pad2): track 0.00 -> 125.4 mm, vias 0 -> 4
- net Net-(SW75-Pad2): track 0.00 -> 125.2 mm, vias 0 -> 4
- net Net-(SW13-Pad2): track 0.00 -> 110.2 mm, vias 0 -> 10
- net Net-(SW2-Pad2): track 0.00 -> 108.7 mm, vias 0 -> 7
- net Net-(SW62-Pad2): track 0.00 -> 108.6 mm, vias 0 -> 6
- net Net-(SW70-Pad2): track 0.00 -> 108.1 mm, vias 0 -> 5
- net Net-(SW38-Pad2): track 0.00 -> 106.5 mm, vias 0 -> 10
- net Net-(SW1-Pad2): track 0.00 -> 102.6 mm
- net Net-(SW81-Pad2): track 0.00 -> 97.1 mm, vias 0 -> 4
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Other:
- board size 309.6 x 123.8 mm -> 312.7 x 138.4 mm

Commit message: Add circuit for the shift registers
Parts:
- added U4: Holyiot-18010-NRF52840, footprints:Holyiot-18010-NRF52840, F.Cu at (292.2, 14.5)
Connections:
- net no_connect_128 renamed no_connect_188
- net no_connect_129 renamed no_connect_189

Commit message: Add circuit for the USB-connector
Parts:
- added D23: PRTR5V0U2X, Package_TO_SOT_SMD:SOT-143, F.Cu at (262.4, 15.3)
- added J1: USB_C_Receptacle_USB2.0, footprints:USB_C_Receptale_JAE_DX07S016JA1R1500, F.Cu at (283.6, 0.66)
- U1: value 74LV595 -> Holyiot-18010-NRF52840; footprint Package_SO:TSSOP-16_4.4x5mm_P0.65mm -> footprints:Holyiot-18010-NRF52840; moved to F.Cu
- U2: value 74LV165 -> 74LV595
- U3: moved to F.Cu
- U4: value Holyiot-18010-NRF52840 -> 74LV165; footprint footprints:Holyiot-18010-NRF52840 -> Package_SO:TSSOP-16_4.4x5mm_P0.65mm
- moved U1 99.8 mm to (216.4, 0.19)
- moved U2 66.8 mm to (252.6, 5.71)
- moved U3 49.9 mm to (252.6, -0.88)
- moved U4 34.4 mm to (261.4, -0.88)
Connections:
- net Net-(U1-Pad14) renamed /VCC_SW_1
- net Net-(U2-Pad7) renamed no_connect_199
- net Net-(U2-Pad9) renamed /595_SERIAL_OUT
- net Net-(U3-Pad7) renamed no_connect_200
- net Net-(U4-Pad10) renamed /165_SERIAL_IN
- net Net-(U4-Pad7) renamed no_connect_201
- U1 pad 1: Net-(D11-Pad3) -> Net-(U1-Pad1)
- U1 pad 15: Net-(D1-Pad3) -> Net-(U1-Pad15)
- U1 pad 16: VCC -> Net-(U1-Pad16)
- U1 pad 2: Net-(D12-Pad3) -> Net-(U1-Pad2)
- U1 pad 3: Net-(D10-Pad3) -> Net-(U1-Pad3)
- U1 pad 4: Net-(D15-Pad3) -> Net-(U1-Pad4)
- U1 pad 5: Net-(D14-Pad3) -> Net-(U1-Pad5)
- U1 pad 6: no_connect_188 -> Net-(U1-Pad6)
- U1 pad 7: no_connect_189 -> Net-(U1-Pad7)
- U1 pad 8: GND -> Net-(U1-Pad8)
- U2 pad 1: Net-(U2-Pad1) -> Net-(D11-Pad3)
- U2 pad 10: Net-(U2-Pad10) -> /VCC_SW
- U2 pad 11: Net-(SW40-Pad2) -> /SPI_SCK
- U2 pad 12: Net-(SW35-Pad2) -> /SPI_SCK
- U2 pad 13: Net-(SW29-Pad2) -> GND
- U2 pad 14: Net-(SW23-Pad2) -> /SPI_MOSI
- U2 pad 15: Net-(U2-Pad15) -> Net-(D1-Pad3)
- U2 pad 16: VCC -> Net-(C4-Pad2)
- U2 pad 2: Net-(U2-Pad2) -> Net-(D12-Pad3)
- U2 pad 3: Net-(SW19-Pad2) -> Net-(D10-Pad3)
- U2 pad 4: Net-(SW13-Pad2) -> Net-(D15-Pad3)
- U2 pad 5: Net-(SW10-Pad2) -> Net-(D14-Pad3)
- U2 pad 6: Net-(SW1-Pad2) -> no_connect_198
- U3 pad 1: Net-(U3-Pad1) -> /165_~PL
- U3 pad 11: Net-(SW81-Pad2) -> Net-(SW40-Pad2)
- U3 pad 12: Net-(SW78-Pad2) -> Net-(SW35-Pad2)
- U3 pad 13: Net-(SW74-Pad2) -> Net-(SW29-Pad2)
- U3 pad 14: Net-(SW68-Pad2) -> Net-(SW23-Pad2)
- U3 pad 15: Net-(U3-Pad15) -> /165_~CE
- U3 pad 16: VCC -> /VCC_SW
- U3 pad 2: Net-(U3-Pad2) -> /SPI_SCK
- U3 pad 3: Net-(SW61-Pad2) -> Net-(SW19-Pad2)
- U3 pad 4: Net-(SW56-Pad2) -> Net-(SW13-Pad2)
- U3 pad 5: Net-(SW51-Pad2) -> Net-(SW10-Pad2)
- U3 pad 6: Net-(SW45-Pad2) -> Net-(SW1-Pad2)
- U3 pad 8: GND -> Net-(C5-Pad1)
- U3 pad 9: Net-(U2-Pad10) -> /SPI_MOSI
- U4 pad 1: Net-(U4-Pad1) -> /165_~PL
- U4 pad 11: Net-(U4-Pad11) -> Net-(SW81-Pad2)
- U4 pad 12: Net-(U4-Pad12) -> Net-(SW78-Pad2)
- U4 pad 13: Net-(U4-Pad13) -> Net-(SW74-Pad2)
- U4 pad 14: Net-(U4-Pad14) -> Net-(SW68-Pad2)
- U4 pad 15: Net-(U4-Pad15) -> /165_~CE
- U4 pad 16: Net-(U4-Pad16) -> /VCC_SW
- U4 pad 2: Net-(U4-Pad2) -> /SPI_SCK
- U4 pad 3: Net-(U4-Pad3) -> Net-(SW61-Pad2)
- U4 pad 4: Net-(U4-Pad4) -> Net-(SW56-Pad2)
- U4 pad 5: Net-(U4-Pad5) -> Net-(SW51-Pad2)
- U4 pad 6: Net-(U4-Pad6) -> Net-(SW45-Pad2)
- U4 pad 9: Net-(U4-Pad9) -> Net-(U3-Pad10)

Commit message: Update the PCB
Parts:
- moved J1 23.7 mm to (298.6, 19.0)
Changed lines of the file:
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@@
   )
   (footprint "footprints:USB_C_Receptale_JAE_DX07S016JA1R1500" (layer "F.Cu")
-    (at 283.6418 0.6604 180)
+    (at 298.577 18.9992 180)
     (property "Dateiname Blatt" "goboard-main.kicad_sch")
     (property "Mouser" " 656-DX07S016JA1R1500 ")
@@
     (fp_line (start -5 5.05) (end 5 5.05) (layer "Dwgs.User") (width 0.12))
     (fp_rect (start -5.22 -2.13) (end 5.22 5.8) (layer "F.CrtYd") (width 0.12) (fill none))
-    (pad "" thru_hole oval (at 4.32 -0.725 180) (size 1.3 2.3) (drill oval 0.6 1.6) (layers *.Cu *.Mask))
-    (pad "" thru_hole oval (at 4.32 3.1 180) (size 1.3 2.6) (drill oval 0.6 1.9) (layers *.Cu *.Mask))
-    (pad "" thru_hole oval (at -4.32 3.1 180) (size 1.3 2.6) (drill oval 0.6 1.9) (layers *.Cu *.Mask))
     (pad "" np_thru_hole oval (at 3.1 0 180) (size 0.85 0.6) (drill oval 0.85 0.6) (layers *.Mask))
-    (pad "" thru_hole oval (at -4.32 -0.725 180) (size 1.3 2.3) (drill oval 0.6 1.6) (layers *.Cu *.Mask))
-    (pad "" smd rect (at -1.4 3.1 180) (size 1 2) (layers "F.Cu" "F.Paste" "F.Mask"))
     (pad "" np_thru_hole circle (at -3.1 0 180) (size 0.6 0.6) (drill 0.6) (layers *.Mask))
-    (pad "" smd rect (at 1.4 3.1 180) (size 1 2) (layers "F.Cu" "F.Paste" "F.Mask"))
     (pad "A1" smd rect (at -3.1 -1.1 180) (size 0.52 1) (layers "F.Cu" "F.Paste" "F.Mask")
       (net 47 "GND") (pinfunction "GND"))
@@
     (pad "B8" smd rect (at -1.25 -1.1 180) (size 0.27 1) (layers "F.Cu" "F.Paste" "F.Mask")
       (net 59 "no_connect_179") (pinfunction "SBU2"))
+    (pad "S1" thru_hole oval (at 4.32 -0.725 180) (size 1.3 2.3) (drill oval 0.6 1.6) (layers *.Cu *.Mask))
+    (pad "S1" smd rect (at -1.4 3.1 180) (size 1 2) (layers "F.Cu" "F.Paste" "F.Mask"))
+    (pad "S1" thru_hole oval (at -4.32 -0.725 180) (size 1.3 2.3) (drill oval 0.6 1.6) (layers *.Cu *.Mask))
+    (pad "S1" thru_hole oval (at -4.32 3.1 180) (size 1.3 2.6) (drill oval 0.6 1.9) (layers *.Cu *.Mask))
+    (pad "S1" thru_hole oval (at 4.32 3.1 180) (size 1.3 2.6) (drill oval 0.6 1.9) (layers *.Cu *.Mask))
+    (pad "S1" smd rect (at 1.4 3.1 180) (size 1 2) (layers "F.Cu" "F.Paste" "F.Mask"))
+    (model "/home/bernd/Dokumente/Projekte-Github/Tastatur/goboard/hardware/3dpackages/DX07S016JA1R1500.3dshapes/DX07S016JA1R1500.wrl"
+      (offset (xyz 0 1.05 1.58))
+      (scale (xyz 1 1 1))
+      (rotate (xyz 0 0 0))
+    )
   )
   (footprint "footprints:SW_Cherry_MX_1.25u_PCB" (layer "F.Cu")

Commit message: Add connector to the numpad to the schematic
Parts:
- moved SW68 37.9 mm to (279.6, 73.8)
- moved SW69 37.9 mm to (279.6, 92.8)
- moved SW73 37.9 mm to (279.6, 169.0)
- moved SW75 37.9 mm to (308.2, 92.8)
- moved SW76 37.9 mm to (315.3, 121.4)
- moved D27 37.9 mm to (224.7, 129.9)
- moved D36 37.9 mm to (284.1, 91.8)
- moved D38 37.9 mm to (298.5, 129.9)
- moved D42 37.9 mm to (331.5, 91.8)
- moved SW10 37.9 mm to (84.3, 130.9)
- moved SW16 37.9 mm to (103.4, 130.9)
- moved SW18 37.9 mm to (77.2, 169.0)
- moved SW22 37.9 mm to (122.4, 130.9)
- moved SW24 37.9 mm to (98.6, 169.0)
- moved SW28 37.9 mm to (141.5, 130.9)
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Routing:
- net Net-(D12-Pad3): track 339.6 -> 267.1 mm, vias 4 -> 0
- net Net-(D11-Pad3): track 308.2 -> 264.9 mm, vias 4 -> 0
- net Net-(D10-Pad3): track 277.1 -> 240.5 mm, vias 2 -> 0
- net Net-(D14-Pad3): track 296.3 -> 274.0 mm
- net Net-(D15-Pad3): track 253.7 -> 236.4 mm

Commit message: Update PCB
Parts:
- added C1: 100nF, Capacitor_SMD:C_0201_0603Metric_Pad0.64x0.40mm_HandSolder, F.Cu at (318.8, 23.0)
- added C2: 4.7nF, Capacitor_SMD:C_0201_0603Metric_Pad0.64x0.40mm_HandSolder, F.Cu at (309.8, 30.1)
- added C3: 100nF, Capacitor_SMD:C_0201_0603Metric_Pad0.64x0.40mm_HandSolder, F.Cu at (340.3, 28.2)
- added C4: 100nF, Capacitor_SMD:C_0201_0603Metric_Pad0.64x0.40mm_HandSolder, F.Cu at (326.8, 23.0)
- added C5: 100nF, Capacitor_SMD:C_0201_0603Metric_Pad0.64x0.40mm_HandSolder, F.Cu at (329.6, 23.0)
- added C6: 100nF, Capacitor_SMD:C_0201_0603Metric_Pad0.64x0.40mm_HandSolder, F.Cu at (326.8, 24.7)
- added C7: 0,1u, Capacitor_SMD:C_0201_0603Metric_Pad0.64x0.40mm_HandSolder, F.Cu at (302.7, 37.7)
- added D45: Power, Diode_SMD:D_0603_1608Metric_Pad1.05x0.95mm_HandSolder, F.Cu at (336.8, 26.0)
- added D46: Caps Lock, Diode_SMD:D_0603_1608Metric_Pad1.05x0.95mm_HandSolder, F.Cu at (341.2, 23.4)
- added D47: Scroll Lock, Diode_SMD:D_0603_1608Metric_Pad1.05x0.95mm_HandSolder, F.Cu at (336.8, 23.4)
- added J2: Conn_02x05_Top_Bottom, Connector_PinSocket_2.54mm:PinSocket_2x05_P2.54mm_Vertical, F.Cu at (306.1, 24.4)
- added J3: Conn_01x01, Connector_PinHeader_2.54mm:PinHeader_1x01_P2.54mm_Vertical, F.Cu at (310.7, 24.4)
- added R1: 0, Resistor_SMD:R_0603_1608Metric_Pad0.98x0.95mm_HandSolder, F.Cu at (315.2, 25.9)
- added R2: 5k1, Resistor_SMD:R_0603_1608Metric_Pad0.98x0.95mm_HandSolder, F.Cu at (310.6, 28.0)
- added R3: 5k1, Resistor_SMD:R_0603_1608Metric_Pad0.98x0.95mm_HandSolder, F.Cu at (315.2, 23.4)
- added R4: 47, Resistor_SMD:R_0603_1608Metric_Pad0.98x0.95mm_HandSolder, F.Cu at (336.7, 28.5)
- added R5: 47, Resistor_SMD:R_0603_1608Metric_Pad0.98x0.95mm_HandSolder, F.Cu at (341.1, 26.0)
- added R6: 47, Resistor_SMD:R_0603_1608Metric_Pad0.98x0.95mm_HandSolder, F.Cu at (336.7, 31.1)
- moved D23 37.3 mm to (311.8, 58.6), turned to 180 degrees
Connections:
- net Net-(U1-Pad10) renamed no_connect_145
- net Net-(U1-Pad11) renamed no_connect_146
- net Net-(U1-Pad12) renamed /UART_RX
- net Net-(U1-Pad18) renamed no_connect_147
- net Net-(U1-Pad19) renamed no_connect_148
- net Net-(U1-Pad2) renamed no_connect_149
- net Net-(U1-Pad20) renamed no_connect_150
- net Net-(U1-Pad26) renamed no_connect_151
- net Net-(U1-Pad3) renamed no_connect_152
- net Net-(U1-Pad33) renamed no_connect_153
- net Net-(U1-Pad34) renamed no_connect_154
- net Net-(U1-Pad35) renamed no_connect_155
- net Net-(U1-Pad36) renamed no_connect_156
- net Net-(U1-Pad4) renamed no_connect_159
- net Net-(U1-Pad5) renamed no_connect_170
- net Net-(U1-Pad6) renamed no_connect_177
- net no_connect_187 renamed no_connect_165
- net no_connect_188 renamed no_connect_166
- net no_connect_189 renamed no_connect_167
- net no_connect_190 renamed no_connect_168
- net no_connect_191 renamed no_connect_169
- net no_connect_192 renamed no_connect_171
- net no_connect_193 renamed no_connect_172
- net no_connect_194 renamed no_connect_173
- net no_connect_195 renamed no_connect_174
- net no_connect_196 renamed no_connect_175
- net no_connect_197 renamed no_connect_176
- J1 pad A8: no_connect_178 -> no_connect_140
- J1 pad B8: no_connect_179 -> no_connect_141
- J1 pad S1: (no net) -> Net-(J1-PadS1)
- U1 pad 1: Net-(U1-Pad1) -> GND
- U1 pad 13: Net-(U1-Pad13) -> /SPI_MISO
- U1 pad 15: Net-(U1-Pad15) -> /165_~CE
- U1 pad 16: Net-(U1-Pad16) -> /SPI_MOSI
- U1 pad 17: Net-(U1-Pad17) -> /165_~PL
- U1 pad 21: Net-(U1-Pad21) -> /RESET
- U1 pad 25: Net-(U1-Pad25) -> GND
- U1 pad 27: Net-(U1-Pad27) -> /SPI_SCK
- U1 pad 31: Net-(U1-Pad31) -> /SWDCLK
- U1 pad 32: Net-(U1-Pad32) -> /SWDIO
- U1 pad 37: Net-(U1-Pad37) -> GND
- U1 pad 38: no_connect_180 -> no_connect_157
- U1 pad 39: no_connect_181 -> no_connect_158
- U1 pad 40: no_connect_182 -> no_connect_160
- U1 pad 41: no_connect_183 -> no_connect_161
- U1 pad 42: no_connect_184 -> no_connect_162
- U1 pad 43: no_connect_185 -> no_connect_163
- U1 pad 44: no_connect_186 -> no_connect_164
- U1 pad 7: Net-(U1-Pad7) -> no_connect_178
- U1 pad 8: Net-(U1-Pad8) -> no_connect_179
- U1 pad 9: Net-(U1-Pad9) -> no_connect_180
- U2 pad 6: no_connect_198 -> no_connect_181
- U2 pad 7: no_connect_199 -> no_connect_182
- U2 pad 9: /595_SERIAL_OUT -> no_connect_183
- U3 pad 7: no_connect_200 -> no_connect_184
- U3 pad 9: /SPI_MOSI -> /SPI_MISO
- U4 pad 10: /165_SERIAL_IN -> no_connect_185
- U4 pad 7: no_connect_201 -> no_connect_186
