File: hardware/main/power.kicad_sch (KiCad schematic)
At the start: 0 parts

Commit message: Add power supply from the debugging connector
The batteries have to be disconnected when the debugger is plugged in,
as the voltages differ (ca. 2V for the batteries, 3.3V for the
debugger).
Parts:
- added BT? (x2): Battery, symbol Device:Battery
- added D?: DIODE, symbol pspice:DIODE
- added Q?: Q_PMOS_DGS, symbol Device:Q_PMOS_DGS
- added R?: R, symbol Device:R
Connections:
- new net: BT?.1 (+), BT?.2 (-)
- new net +3V3: D?.1 (K), Q?.2 (G), R?.1
- new net +BATT: Q?.1 (D)
- new net GND: R?.2
- new net VCC_SW: D?.2 (A), Q?.3 (S)
Other:
- note added: "TODO: Difference between 3,3V and V_Batt has to be greater than Vgs"
- note added: "TODO: The diode has to be one with very little voltage drop otherwise the microcontroller may not program correctly"
- note added: "TODO: add jumpers as a precaution if this does not work"
Changed lines of the file:
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@@
 (kicad_sch (version 20201015) (generator eeschema)
   (paper "A4")
+  (junction (at 81.28 124.46) (diameter 1.016) (color 0 0 0 0))
+  (junction (at 83.82 124.46) (diameter 1.016) (color 0 0 0 0))
+  (junction (at 93.98 139.7) (diameter 1.016) (color 0 0 0 0))
+  (wire (pts (xy 72.39 124.46) (xy 72.39 127))
+    (stroke (width 0) (type solid) (color 0 0 0 0))
+  )
+  (wire (pts (xy 72.39 124.46) (xy 81.28 124.46))
+    (stroke (width 0) (type solid) (color 0 0 0 0))
+  )
+  (wire (pts (xy 72.39 134.62) (xy 72.39 137.16))
+    (stroke (width 0) (type solid) (color 0 0 0 0))
+  )
+  (wire (pts (xy 74.93 93.98) (xy 80.01 93.98))
+    (stroke (width 0) (type solid) (color 0 0 0 0))
+  )
+  (wire (pts (xy 81.28 121.92) (xy 81.28 124.46))
+    (stroke (width 0) (type solid) (color 0 0 0 0))
+  )
+  (wire (pts (xy 81.28 124.46) (xy 83.82 124.46))
+    (stroke (width 0) (type solid) (color 0 0 0 0))
+  )
+  (wire (pts (xy 83.82 124.46) (xy 83.82 127))
+    (stroke (width 0) (type solid) (color 0 0 0 0))
+  )
+  (wire (pts (xy 83.82 124.46) (xy 86.36 124.46))
+    (stroke (width 0) (type solid) (color 0 0 0 0))
+  )
+  (wire (pts (xy 83.82 137.16) (xy 83.82 139.7))
+    (stroke (width 0) (type solid) (color 0 0 0 0))
+  )
+  (wire (pts (xy 83.82 139.7) (xy 93.98 139.7))
+    (stroke (width 0) (type solid) (color 0 0 0 0))
+  )
+  (wire (pts (xy 90.17 93.98) (xy 95.25 93.98))
+    (stroke (width 0) (type solid) (color 0 0 0 0))
+  )
+  (wire (pts (xy 93.98 116.84) (xy 93.98 119.38))
+    (stroke (width 0) (type solid) (color 0 0 0 0))
+  )
+  (wire (pts (xy 93.98 139.7) (xy 93.98 129.54))
+    (stroke (width 0) (type solid) (color 0 0 0 0))
+  )
+  (wire (pts (xy 93.98 139.7) (xy 111.76 139.7))
+    (stroke (width 0) (type solid) (color 0 0 0 0))
+  )
+  (wire (pts (xy 111.76 137.16) (xy 111.76 139.7))
+    (stroke (width 0) (type solid) (color 0 0 0 0))
+  )
+  (text "TODO: add jumpers as a precaution if this does not work"
+    (at 49.53 149.86 0)
+    (effects (font (size 1.27 1.27)) (justify left bottom))
+  )
+  (text "TODO: Difference between 3,3V and\nV_Batt has to be greater than Vgs"
+    (at 120.65 121.92 0)
+    (effects (font (size 1.27 1.27)) (justify left bottom))
+  )
+  (text "TODO: The diode has to be one with very little voltage drop\notherwise the microcontroller may not program correctly"
+    (at 120.65 128.27 0)
+    (effects (font (size 1.27 1.27)) (justify left bottom))
+  )
+  (hierarchical_label "VCC_SW" (shape input) (at 111.76 137.16 90)
+    (effects (font (size 1.27 1.27)) (justify left))
+  )
+  (symbol (lib_id "power:+5V") (at 40.64 34.29 0) (unit 1)
+    (in_bom yes) (on_board yes)
+    (property "Reference" "#PWR?" (id 0) (at 40.64 38.1 0)
+      (effects (font (size 1.27 1.27)) hide)
+    )
+    (property "Value" "+5V" (id 1) (at 41.0083 29.9656 0))
+    (property "Footprint" "" (id 2) (at 40.64 34.29 0)
+      (effects (font (size 1.27 1.27)) hide)
+    )
+    (property "Datasheet" "" (id 3) (at 40.64 34.29 0)
+      (effects (font (size 1.27 1.27)) hide)
+    )
+  )
+  (symbol (lib_id "power:+3.3V") (at 81.28 121.92 0) (unit 1)
+    (in_bom yes) (on_board yes)
+    (property "Reference" "#PWR?" (id 0) (at 81.28 125.73 0)
+      (effects (font (size 1.27 1.27)) hide)
+    )
+    (property "Value" "+3.3V_programmer" (id 1) (at 81.648 117.596 0))
+    (property "Footprint" "" (id 2) (at 81.28 121.92 0)
+      (effects (font (size 1.27 1.27)) hide)
+    )
+    (property "Datasheet" "" (id 3) (at 81.28 121.92 0)
+      (effects (font (size 1.27 1.27)) hide)
+    )
+  )
+  (symbol (lib_id "power:+BATT") (at 93.98 116.84 0) (unit 1)
+    (in_bom yes) (on_board yes)
+    (property "Reference" "#PWR?" (id 0) (at 93.98 120.65 0)
+      (effects (font (size 1.27 1.27)) hide)
+    )
+    (property "Value" "+BATT" (id 1) (at 94.3483 112.5156 0))
+    (property "Footprint" "" (id 2) (at 93.98 116.84 0)
+      (effects (font (size 1.27 1.27)) hide)
+    )
+    (property "Datasheet" "" (id 3) (at 93.98 116.84 0)
+      (effects (font (size 1.27 1.27)) hide)
+    )
+  )
+  (symbol (lib_id "power:GND") (at 72.39 137.16 0) (unit 1)
+    (in_bom yes) (on_board yes)
+    (property "Reference" "#PWR?" (id 0) (at 72.39 143.51 0)
+      (effects (font (size 1.27 1.27)) hide)
+    )
+    (property "Value" "GND" (id 1) (at 72.5043 141.4844 0))
+    (property "Footprint" "" (id 2) (at 72.39 137.16 0)
+      (effects (font (size 1.27 1.27)) hide)
+    )
+    (property "Datasheet" "" (id 3) (at 72.39 137.16 0)
+      (effects (font (size 1.27 1.27)) hide)
+    )
+  )
+  (symbol (lib_id "Device:R") (at 72.39 130.81 0) (unit 1)
+    (in_bom yes) (on_board yes)
+    (property "Reference" "R?" (id 0) (at 74.1681 129.6606 0)
+      (effects (font (size 1.27 1.27)) (justify left))
+    )
+    (property "Value" "R" (id 1) (at 74.1681 131.9593 0)
+      (effects (font (size 1.27 1.27)) (justify left))
+    )
+    (property "Footprint" "" (id 2) (at 70.612 130.81 90)
+      (effects (font (size 1.27 1.27)) hide)
+    )
+    (property "Datasheet" "~" (id 3) (at 72.39 130.81 0)
+      (effects (font (size 1.27 1.27)) hide)
+    )
+  )
+  (symbol (lib_id "Device:Battery") (at 69.85 93.98 90) (unit 1)
+    (in_bom yes) (on_board yes)
+    (property "Reference" "BT?" (id 0) (at 69.85 87.8648 90))
+    (property "Value" "Battery" (id 1) (at 69.85 90.1635 90))
+    (property "Footprint" "" (id 2) (at 68.326 93.98 90)
+      (effects (font (size 1.27 1.27)) hide)
+    )
+    (property "Datasheet" "~" (id 3) (at 68.326 93.98 90)
+      (effects (font (size 1.27 1.27)) hide)
+    )
+  )
+  (symbol (lib_id "Device:Battery") (at 85.09 93.98 90) (unit 1)
+    (in_bom yes) (on_board yes)
+    (property "Reference" "BT?" (id 0) (at 85.09 87.8648 90))
+    (property "Value" "Battery" (id 1) (at 85.09 90.1635 90))
+    (property "Footprint" "" (id 2) (at 83.566 93.98 90)
+      (effects (font (size 1.27 1.27)) hide)
+    )
+    (property "Datasheet" "~" (id 3) (at 83.566 93.98 90)
+      (effects (font (size 1.27 1.27)) hide)
+    )
+  )
+  (symbol (lib_id "pspice:DIODE") (at 83.82 132.08 270) (unit 1)
+    (in_bom yes) (on_board yes)
+    (property "Reference" "D?" (id 0) (at 86.9951 130.9306 90)
+      (effects (font (size 1.27 1.27)) (justify left))
+    )
+    (property "Value" "DIODE" (id 1) (at 86.9951 133.2293 90)
+      (effects (font (size 1.27 1.27)) (justify left))
+    )
+    (property "Footprint" "" (id 2) (at 83.82 132.08 0)
+      (effects (font (size 1.27 1.27)) hide)
+    )
+    (property "Datasheet" "~" (id 3) (at 83.82 132.08 0)
+      (effects (font (size 1.27 1.27)) hide)
+    )
+  )
+  (symbol (lib_id "Device:Q_PMOS_DGS") (at 91.44 124.46 0) (unit 1)
+    (in_bom yes) (on_board yes)
+    (property "Reference" "Q?" (id 0) (at 96.6471 123.3106 0)
+      (effects (font (size 1.27 1.27)) (justify left))
+    )
+    (property "Value" "Q_PMOS_DGS" (id 1) (at 96.6471 125.6093 0)
+      (effects (font (size 1.27 1.27)) (justify left))
+    )
+    (property "Footprint" "" (id 2) (at 96.52 121.92 0)
+      (effects (font (size 1.27 1.27)) hide)
+    )
+    (property "Datasheet" "~" (id 3) (at 91.44 124.46 0)
+      (effects (font (size 1.27 1.27)) hide)
+    )
+  )
 )
