File: hardware/main/keys.kicad_sch (KiCad schematic)
At the start: 134 parts, among them SW1 Esc, SW10 a, SW12 Fn, SW13 F2, SW14 2, SW15 w, SW16 s, SW17 z, SW18 Tux, SW19 F3, SW2 F1, SW20 3, SW21 e, SW22 d, SW23 c, SW24 Alt, SW25 F4, SW26 4, SW27 r, SW28 f, SW29 v, SW3 tilde, SW31 F5, SW32 5, SW33 t, SW34 g, SW35 b, SW36 F6, SW37 6, SW38 y, SW39 h, SW4 Tab, SW40 n, SW41 F7, SW42 7, SW43 u, SW44 j, SW45 m, SW46 Space, SW47 F8, SW48 8, SW49 i, SW5 Caps Lock, SW50 k, SW51 ,, SW52 F9, SW53 9, SW54 o, SW55 l, SW56 ., SW57 F10, SW58 0, SW59 p, SW6 Shift, SW60 ;, SW61 /, SW62 Alt Gr, SW63 F11, SW64 -, SW65 [, SW66 ', SW67 Menu, SW68 F12, SW69 =, SW7 Ctrl, SW70 ], SW71 \, SW72 Shift, SW73 Ctrl, SW74 Print, SW75 Backspace, SW76 Enter, SW77 Left, SW78 Scroll Lock, SW79 Up, SW8 1, SW80 Down, SW81 Pause, SW82 INS, SW83 DEL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

Commit message: Adapt the layout for another keycap set
The layout is now compatible with this keycap set:
https://hk-gaming.com/collections/keycaps/products/hk-gaming-dye-
sublimation-cherry-profile-thick-pbt-keysets-for-mechanical-keyboard-139
-keys-chalk
Parts:
- removed SW67: Menu, footprints:SW_Cherry_MX_1.00u_PCB, symbol Switch:SW_Push_45deg
- SW24: footprint footprints:SW_Cherry_MX_1.00u_PCB -> footprints:SW_Cherry_MX_1.25u_PCB
- SW62: footprint footprints:SW_Cherry_MX_1.25u_PCB -> footprints:SW_Cherry_MX_1.50u_PCB
- SW73: footprint footprints:SW_Cherry_MX_1.00u_PCB -> footprints:SW_Cherry_MX_1.50u_PCB
Connections:
- net at SW61.2, SW63.2, SW64.2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: now also SW73.2
- net at SW73.1: now also D34.1; no longer D40.2
- net at SW68.2, SW69.2, SW70.2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: now also SW77.2; no longer SW73.2
- net at D40.1: no longer SW77.1
- net at SW74.2, SW75.2, SW76.2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: no longer SW77.2
- new net: D40.2, SW77.1
- no-connect marks 6 -> 7
Other:
- moved on the sheet: SW73, SW77
Changed lines of the file:
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@@
   (junction (at 330.2 78.74) (diameter 1.016) (color 0 0 0 0))
   (junction (at 330.2 104.14) (diameter 1.016) (color 0 0 0 0))
-  (junction (at 330.2 180.34) (diameter 1.016) (color 0 0 0 0))
   (junction (at 355.6 78.74) (diameter 1.016) (color 0 0 0 0))
   (junction (at 355.6 154.94) (diameter 1.016) (color 0 0 0 0))
@@
   (junction (at 365.76 154.94) (diameter 1.016) (color 0 0 0 0))
   (junction (at 365.76 180.34) (diameter 1.016) (color 0 0 0 0))
-  (no_connect (at 60.96 71.12))
+  (no_connect (at 317.5 162.56))
   (no_connect (at 269.24 208.28))
+  (no_connect (at 60.96 76.2))
+  (no_connect (at 124.46 233.68))
   (no_connect (at 60.96 68.58))
   (no_connect (at 266.7 233.68))
-  (no_connect (at 60.96 76.2))
-  (no_connect (at 124.46 233.68))
+  (no_connect (at 60.96 71.12))
   (wire (pts (xy 25.4 58.42) (xy 27.94 58.42))
     (stroke (width 0) (type solid) (color 0 0 0 0))
@@
     (stroke (width 0) (type solid) (color 0 0 0 0))
   )
+  (wire (pts (xy 281.94 162.56) (xy 287.02 162.56))
+    (stroke (width 0) (type solid) (color 0 0 0 0))
+  )
   (wire (pts (xy 284.48 53.34) (xy 284.48 78.74))
     (stroke (width 0) (type solid) (color 0 0 0 0))
@@
     (stroke (width 0) (type solid) (color 0 0 0 0))
   )
-  (wire (pts (xy 287.02 162.56) (xy 281.94 162.56))
-    (stroke (width 0) (type solid) (color 0 0 0 0))
-  )
-  (wire (pts (xy 287.02 175.26) (xy 287.02 162.56))
+  (wire (pts (xy 287.02 162.56) (xy 287.02 175.26))
     (stroke (width 0) (type solid) (color 0 0 0 0))
   )
@@
     (stroke (width 0) (type solid) (color 0 0 0 0))
   )
-  (wire (pts (xy 322.58 162.56) (xy 317.5 162.56))
-    (stroke (width 0) (type solid) (color 0 0 0 0))
-  )
-  (wire (pts (xy 322.58 162.56) (xy 322.58 175.26))
-    (stroke (width 0) (type solid) (color 0 0 0 0))
-  )
   (wire (pts (xy 327.66 53.34) (xy 330.2 53.34))
     (stroke (width 0) (type solid) (color 0 0 0 0))
@@
     (stroke (width 0) (type solid) (color 0 0 0 0))
   )
-  (wire (pts (xy 327.66 180.34) (xy 330.2 180.34))
-    (stroke (width 0) (type solid) (color 0 0 0 0))
-  )
   (wire (pts (xy 330.2 53.34) (xy 330.2 78.74))
     (stroke (width 0) (type solid) (color 0 0 0 0))
@@
     (stroke (width 0) (type solid) (color 0 0 0 0))
   )
-  (wire (pts (xy 330.2 104.14) (xy 330.2 180.34))
-    (stroke (width 0) (type solid) (color 0 0 0 0))
-  )
-  (wire (pts (xy 330.2 180.34) (xy 330.2 198.12))
+  (wire (pts (xy 330.2 104.14) (xy 330.2 198.12))
     (stroke (width 0) (type solid) (color 0 0 0 0))
   )
@@
     (property "Reference" "SW24" (id 0) (at 127 170.7958 0))
     (property "Value" "Alt" (id 1) (at 127 173.095 0))
-    (property "Footprint" "footprints:SW_Cherry_MX_1.00u_PCB" (id 2) (at 127 177.8 0)
+    (property "Footprint" "footprints:SW_Cherry_MX_1.25u_PCB" (id 2) (at 127 177.8 0)
       (effects (font (size 1.27 1.27)) hide)
     )
@@
     (property "Reference" "SW62" (id 0) (at 269.24 170.7958 0))
     (property "Value" "Alt Gr" (id 1) (at 269.24 173.095 0))
-    (property "Footprint" "footprints:SW_Cherry_MX_1.25u_PCB" (id 2) (at 269.24 177.8 0)
+    (property "Footprint" "footprints:SW_Cherry_MX_1.50u_PCB" (id 2) (at 269.24 177.8 0)
       (effects (font (size 1.27 1.27)) hide)
     )
@@
   (symbol (lib_id "Switch:SW_Push_45deg") (at 289.56 177.8 0) (unit 1)
     (in_bom yes) (on_board yes)
-    (property "Reference" "SW67" (id 0) (at 289.56 170.7958 0))
-    (property "Value" "Menu" (id 1) (at 289.56 173.095 0))
-    (property "Footprint" "footprints:SW_Cherry_MX_1.00u_PCB" (id 2) (at 289.56 177.8 0)
+    (property "Reference" "SW73" (id 0) (at 289.56 170.7958 0))
+    (property "Value" "Ctrl" (id 1) (at 289.56 173.095 0))
+    (property "Footprint" "footprints:SW_Cherry_MX_1.50u_PCB" (id 2) (at 289.56 177.8 0)
       (effects (font (size 1.27 1.27)) hide)
     )
@@
   (symbol (lib_id "Switch:SW_Push_45deg") (at 304.8 177.8 0) (unit 1)
     (in_bom yes) (on_board yes)
-    (property "Reference" "SW73" (id 0) (at 304.8 170.7958 0))
-    (property "Value" "Ctrl" (id 1) (at 304.8 173.095 0))
+    (property "Reference" "SW77" (id 0) (at 304.8 170.7958 0))
+    (property "Value" "Left" (id 1) (at 304.8 173.095 0))
     (property "Footprint" "footprints:SW_Cherry_MX_1.00u_PCB" (id 2) (at 304.8 177.8 0)
       (effects (font (size 1.27 1.27)) hide)
@@
       (effects (font (size 1.27 1.27)) hide)
     )
-  )
-  (symbol (lib_id "Switch:SW_Push_45deg") (at 325.12 177.8 0) (unit 1)
-    (in_bom yes) (on_board yes)
-    (property "Reference" "SW77" (id 0) (at 325.12 170.7958 0))
-    (property "Value" "Left" (id 1) (at 325.12 173.095 0))
-    (property "Footprint" "footprints:SW_Cherry_MX_1.00u_PCB" (id 2) (at 325.12 177.8 0)
-      (effects (font (size 1.27 1.27)) hide)
-    )
-    (property "Datasheet" "https://www.mouser.de/datasheet/2/71/EN_CHERRY_MX_BLUE-1608304.pdf" (id 3) (at 325.12 177.8 0)
-      (effects (font (size 1.27 1.27)) hide)
-    )
-    (property "Mouser" "540-MX1A-E1NW" (id 4) (at 325.12 177.8 0)
-      (effects (font (size 1.27 1.27)) hide)
-    )
-    (property "Part Name" "MX1A-E1NW" (id 5) (at 325.12 177.8 0)
-      (effects (font (size 1.27 1.27)) hide)
-    )

Commit message: Fix footprint of the capacitors
Parts:
- C4, C5, C6: footprint Capacitor_SMD:C_0201_0603Metric_Pad0.64x0.40mm_HandSolder -> Capacitor_SMD:C_0603_1608Metric_Pad1.08x0.95mm_HandSolder
Changed lines of the file:
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@@
       (effects (font (size 1.27 1.27)) (justify left))
     )
-    (property "Footprint" "Capacitor_SMD:C_0201_0603Metric_Pad0.64x0.40mm_HandSolder" (id 2) (at 59.3852 48.26 0)
+    (property "Footprint" "Capacitor_SMD:C_0603_1608Metric_Pad1.08x0.95mm_HandSolder" (id 2) (at 59.3852 48.26 0)
       (effects (font (size 1.27 1.27)) hide)
     )
@@
       (effects (font (size 1.27 1.27)) (justify left))
     )
-    (property "Footprint" "Capacitor_SMD:C_0201_0603Metric_Pad0.64x0.40mm_HandSolder" (id 2) (at 80.9752 228.6 0)
+    (property "Footprint" "Capacitor_SMD:C_0603_1608Metric_Pad1.08x0.95mm_HandSolder" (id 2) (at 80.9752 228.6 0)
       (effects (font (size 1.27 1.27)) hide)
     )
@@
       (effects (font (size 1.27 1.27)) (justify left))
     )
-    (property "Footprint" "Capacitor_SMD:C_0201_0603Metric_Pad0.64x0.40mm_HandSolder" (id 2) (at 223.2152 228.6 0)
+    (property "Footprint" "Capacitor_SMD:C_0603_1608Metric_Pad1.08x0.95mm_HandSolder" (id 2) (at 223.2152 228.6 0)
       (effects (font (size 1.27 1.27)) hide)
     )

Commit message: Change value field for the backslash-key
The value "\" caused the FreeCAD-StepUp load to fail due to a parsing
error.
Parts:
- SW71: value \ -> backslash
Changed lines of the file:
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@@
     (in_bom yes) (on_board yes)
     (property "Reference" "SW71" (id 0) (at 304.8 119.9958 0))
-    (property "Value" "\\" (id 1) (at 304.8 122.295 0))
+    (property "Value" "backslash" (id 1) (at 304.8 122.295 0))
     (property "Footprint" "footprints:SW_Cherry_MX_1.00u_PCB" (id 2) (at 304.8 127 0)
       (effects (font (size 1.27 1.27)) hide)

Commit message: Write out the symbol names for the keys
Parts:
- SW51: value , -> comma
- SW56: value . -> dot
- SW60: value ; -> semicolon
- SW61: value / -> slash
- SW64: value - -> minus
- SW65: value [ -> sq br open
- SW66: value ' -> apostrophe
- SW69: value = -> equal
- SW70: value ] -> sq br close
Changed lines of the file:
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@@
     (in_bom yes) (on_board yes)
     (property "Reference" "SW51" (id 0) (at 254 145.3958 0))
-    (property "Value" "," (id 1) (at 254 147.695 0))
+    (property "Value" "comma" (id 1) (at 254 147.695 0))
     (property "Footprint" "footprints:SW_Cherry_MX_1.00u_PCB" (id 2) (at 254 152.4 0)
       (effects (font (size 1.27 1.27)) hide)
@@
     (in_bom yes) (on_board yes)
     (property "Reference" "SW60" (id 0) (at 269.24 119.9958 0))
-    (property "Value" ";" (id 1) (at 269.24 122.295 0))
+    (property "Value" "semicolon" (id 1) (at 269.24 122.295 0))
     (property "Footprint" "footprints:SW_Cherry_MX_1.00u_PCB" (id 2) (at 269.24 127 0)
       (effects (font (size 1.27 1.27)) hide)
@@
     (in_bom yes) (on_board yes)
     (property "Reference" "SW56" (id 0) (at 269.24 145.3958 0))
-    (property "Value" "." (id 1) (at 269.24 147.695 0))
+    (property "Value" "dot" (id 1) (at 269.24 147.695 0))
     (property "Footprint" "footprints:SW_Cherry_MX_1.00u_PCB" (id 2) (at 269.24 152.4 0)
       (effects (font (size 1.27 1.27)) hide)
@@
     (in_bom yes) (on_board yes)
     (property "Reference" "SW64" (id 0) (at 289.56 69.1958 0))
-    (property "Value" "-" (id 1) (at 289.56 71.495 0))
+    (property "Value" "minus" (id 1) (at 289.56 71.495 0))
     (property "Footprint" "footprints:SW_Cherry_MX_1.00u_PCB" (id 2) (at 289.56 76.2 0)
       (effects (font (size 1.27 1.27)) hide)
@@
     (in_bom yes) (on_board yes)
     (property "Reference" "SW65" (id 0) (at 289.56 94.5958 0))
-    (property "Value" "[" (id 1) (at 289.56 96.895 0))
+    (property "Value" "sq br open" (id 1) (at 289.56 96.895 0))
     (property "Footprint" "footprints:SW_Cherry_MX_1.00u_PCB" (id 2) (at 289.56 101.6 0)
       (effects (font (size 1.27 1.27)) hide)
@@
     (in_bom yes) (on_board yes)
     (property "Reference" "SW66" (id 0) (at 289.56 119.9958 0))
-    (property "Value" "'" (id 1) (at 289.56 122.295 0))
+    (property "Value" "apostrophe" (id 1) (at 289.56 122.295 0))
     (property "Footprint" "footprints:SW_Cherry_MX_1.00u_PCB" (id 2) (at 289.56 127 0)
       (effects (font (size 1.27 1.27)) hide)
@@
     (in_bom yes) (on_board yes)
     (property "Reference" "SW61" (id 0) (at 289.56 145.3958 0))
-    (property "Value" "/" (id 1) (at 289.56 147.695 0))
+    (property "Value" "slash" (id 1) (at 289.56 147.695 0))
     (property "Footprint" "footprints:SW_Cherry_MX_1.00u_PCB" (id 2) (at 289.56 152.4 0)
       (effects (font (size 1.27 1.27)) hide)
@@
     (in_bom yes) (on_board yes)
     (property "Reference" "SW69" (id 0) (at 304.8 69.1958 0))
-    (property "Value" "=" (id 1) (at 304.8 71.495 0))
+    (property "Value" "equal" (id 1) (at 304.8 71.495 0))
     (property "Footprint" "footprints:SW_Cherry_MX_1.00u_PCB" (id 2) (at 304.8 76.2 0)
       (effects (font (size 1.27 1.27)) hide)
@@
     (in_bom yes) (on_board yes)
     (property "Reference" "SW70" (id 0) (at 304.8 94.5958 0))
-    (property "Value" "]" (id 1) (at 304.8 96.895 0))
+    (property "Value" "sq br close" (id 1) (at 304.8 96.895 0))
     (property "Footprint" "footprints:SW_Cherry_MX_1.00u_PCB" (id 2) (at 304.8 101.6 0)
       (effects (font (size 1.27 1.27)) hide)

Commit message: Revert to a key layout with a menu key between alt gr and ctrl
Parts:
- added SW?: Menu, footprints:SW_Cherry_MX_1.00u_PCB, symbol Switch:SW_Push_45deg
- SW62, SW73: footprint footprints:SW_Cherry_MX_1.50u_PCB -> footprints:SW_Cherry_MX_1.00u_PCB
Connections:
- net at SW61.2, SW63.2, SW64.2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: now also SW?.2; no longer SW73.2
- net at SW73.1: now also D40.2; no longer D34.1
- net at SW68.2, SW69.2, SW70.2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: now also SW73.2; no longer SW77.2
- net at D40.1: now also SW77.1
- net at SW74.2, SW75.2, SW76.2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: now also SW77.2
- new net: D34.1, SW?.1
- no-connect marks 7 -> 6
Other:
- moved on the sheet: SW73, SW77
Changed lines of the file:
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@@
   (junction (at 330.2 78.74) (diameter 1.016) (color 0 0 0 0))
   (junction (at 330.2 104.14) (diameter 1.016) (color 0 0 0 0))
+  (junction (at 330.2 180.34) (diameter 1.016) (color 0 0 0 0))
   (junction (at 355.6 78.74) (diameter 1.016) (color 0 0 0 0))
   (junction (at 355.6 154.94) (diameter 1.016) (color 0 0 0 0))
@@
   (no_connect (at 266.7 233.68))
   (no_connect (at 269.24 208.28))
-  (no_connect (at 317.5 162.56))
   (wire (pts (xy 25.4 58.42) (xy 27.94 58.42))
     (stroke (width 0) (type solid) (color 0 0 0 0))
@@
     (stroke (width 0) (type solid) (color 0 0 0 0))
   )
+  (wire (pts (xy 317.5 162.56) (xy 322.58 162.56))
+    (stroke (width 0) (type solid) (color 0 0 0 0))
+  )
   (wire (pts (xy 320.04 53.34) (xy 320.04 78.74))
     (stroke (width 0) (type solid) (color 0 0 0 0))
@@
     (stroke (width 0) (type solid) (color 0 0 0 0))
   )
+  (wire (pts (xy 322.58 162.56) (xy 322.58 175.26))
+    (stroke (width 0) (type solid) (color 0 0 0 0))
+  )
   (wire (pts (xy 327.66 53.34) (xy 330.2 53.34))
     (stroke (width 0) (type solid) (color 0 0 0 0))
@@
     (stroke (width 0) (type solid) (color 0 0 0 0))
   )
+  (wire (pts (xy 327.66 180.34) (xy 330.2 180.34))
+    (stroke (width 0) (type solid) (color 0 0 0 0))
+  )
   (wire (pts (xy 330.2 53.34) (xy 330.2 78.74))
     (stroke (width 0) (type solid) (color 0 0 0 0))
@@
     (stroke (width 0) (type solid) (color 0 0 0 0))
   )
-  (wire (pts (xy 330.2 104.14) (xy 330.2 198.12))
+  (wire (pts (xy 330.2 104.14) (xy 330.2 180.34))
+    (stroke (width 0) (type solid) (color 0 0 0 0))
+  )
+  (wire (pts (xy 330.2 180.34) (xy 330.2 198.12))
     (stroke (width 0) (type solid) (color 0 0 0 0))
   )
@@
     (property "Reference" "SW62" (id 0) (at 269.24 170.7958 0))
     (property "Value" "Alt Gr" (id 1) (at 269.24 173.095 0))
-    (property "Footprint" "footprints:SW_Cherry_MX_1.50u_PCB" (id 2) (at 269.24 177.8 0)
+    (property "Footprint" "footprints:SW_Cherry_MX_1.00u_PCB" (id 2) (at 269.24 177.8 0)
       (effects (font (size 1.27 1.27)) hide)
     )
@@
   (symbol (lib_id "Switch:SW_Push_45deg") (at 289.56 177.8 0) (unit 1)
     (in_bom yes) (on_board yes)
-    (property "Reference" "SW73" (id 0) (at 289.56 170.7958 0))
-    (property "Value" "Ctrl" (id 1) (at 289.56 173.095 0))
-    (property "Footprint" "footprints:SW_Cherry_MX_1.50u_PCB" (id 2) (at 289.56 177.8 0)
+    (property "Reference" "SW?" (id 0) (at 289.56 170.7958 0))
+    (property "Value" "Menu" (id 1) (at 289.56 173.095 0))
+    (property "Footprint" "footprints:SW_Cherry_MX_1.00u_PCB" (id 2) (at 289.56 177.8 0)
       (effects (font (size 1.27 1.27)) hide)
     )
@@
   (symbol (lib_id "Switch:SW_Push_45deg") (at 304.8 177.8 0) (unit 1)
     (in_bom yes) (on_board yes)
-    (property "Reference" "SW77" (id 0) (at 304.8 170.7958 0))
-    (property "Value" "Left" (id 1) (at 304.8 173.095 0))
+    (property "Reference" "SW73" (id 0) (at 304.8 170.7958 0))
+    (property "Value" "Ctrl" (id 1) (at 304.8 173.095 0))
     (property "Footprint" "footprints:SW_Cherry_MX_1.00u_PCB" (id 2) (at 304.8 177.8 0)
       (effects (font (size 1.27 1.27)) hide)
@@
       (effects (font (size 1.27 1.27)) hide)
     )
+  )
+  (symbol (lib_id "Switch:SW_Push_45deg") (at 325.12 177.8 0) (unit 1)
+    (in_bom yes) (on_board yes)
+    (property "Reference" "SW77" (id 0) (at 325.12 170.7958 0))
+    (property "Value" "Left" (id 1) (at 325.12 173.095 0))
+    (property "Footprint" "footprints:SW_Cherry_MX_1.00u_PCB" (id 2) (at 325.12 177.8 0)
+      (effects (font (size 1.27 1.27)) hide)
+    )
+    (property "Datasheet" "https://www.mouser.de/datasheet/2/71/EN_CHERRY_MX_BLUE-1608304.pdf" (id 3) (at 325.12 177.8 0)
+      (effects (font (size 1.27 1.27)) hide)
+    )
+    (property "Mouser" "540-MX1A-E1NW" (id 4) (at 325.12 177.8 0)
+      (effects (font (size 1.27 1.27)) hide)
+    )
+    (property "Part Name" "MX1A-E1NW" (id 5) (at 325.12 177.8 0)
+      (effects (font (size 1.27 1.27)) hide)
+    )
